File: TKL_Keyboard.kicad_pcb (KiCad board)
At the start: 2 copper layers, 372.7 x 125 mm, 214 parts, among them J1 USB_C_Receptacle_USB2.0, J2 Conn_01x05_Male, SW2 RotaryEncoder_Switch, SW3 SW_SPDT, U2 XC6206PxxxMR, U4 STM32F303C8Tx, Y1 8MHz

Commit message: small changes
Small Changes

Small Changes

Small Changes

Small Changes

Small Changes

small changes
Parts:
- added G***: LOGO, LOGO, F.Cu at (346.8, 112.8)
- added R6: 10k, Resistor_SMD:R_0805_2012Metric, B.Cu at (47.8, 48.5)
- added R8: 10k, Resistor_SMD:R_0805_2012Metric, B.Cu at (45.8, 49.9)
- C1: renamed from C97; value 1uF -> 22uF; footprint Capacitor_SMD:C_0402_1005Metric -> Capacitor_SMD:C_0805_2012Metric
- C2: renamed from C98; value 1uF -> 22uF; footprint Capacitor_SMD:C_0402_1005Metric -> Capacitor_SMD:C_0805_2012Metric
- C3: renamed from C99; value 30p -> 30pF
- C4: renamed from C100; value 30p -> 30pF
- MX31: footprint MX_Only:MXOnly-1U-Hotswap -> MX_Only:MXOnly-2U-Hotswap
- R1, R2: moved to B.Cu
- Y1: value 8MHz -> 16MHz
- moved C14 34.3 mm to (66.8, 45.1)
- moved C15 31.1 mm to (68.5, 47.3)
- moved R2 9.16 mm to (92.9, 29.6), turned to 0 degrees
- moved C11 2.55 mm to (75.6, 51.5), turned to 90 degrees
- moved FB1 1.79 mm to (74.3, 52.8), turned to 90 degrees
- moved R5 1.14 mm to (93.9, 48.8), turned to 0 degrees
- moved R1 0.80 mm to (80.4, 36.0)
- moved C2 0.55 mm to (78.2, 36.9)
- moved C12 0.54 mm to (75.6, 54.1)
- moved C1 0.51 mm to (75.0, 34.2)
- moved MX50 0.29 mm to (352.2, 85.6)
- moved MX34 0.27 mm to (390.3, 66.5)
- moved R7 0.25 mm to (84.0, 36.8)
- moved MX10 0.24 mm to (271.3, 38.0)
- moved MX29 0.24 mm to (271.3, 66.5)
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- renumbered C105 to C10, C104 to C11, C108 to C12, C107 to C13, C101 to C14, C102 to C15, C106 to C5, C86 to C6, C94 to C7, C95 to C8, C96 to C9, R5 to R3, R6 to R4, R7 to R5, R8 to R7, SW3 to SW1
Connections:
- C12 pad 1: Net-(C108-Pad1) -> +3V3
- C13 pad 1: NRST -> GND
- C13 pad 2: GND -> NRST
- C14 pad 1: Net-(C101-Pad1) -> ENCODER_A
- C15 pad 1: Net-(C102-Pad1) -> ENCODER_B
- D34 pad 2: unconnected-(D34-A-Pad2) -> Net-(D34-A)
- FB1 pad 1: Net-(C108-Pad1) -> +3V3
- J1 pad A6: USB_CON_D- -> USB_CON_D+
- J1 pad A7: USB_CON_D+ -> USB_CON_D-
- J1 pad B6: USB_CON_D- -> USB_CON_D+
- J1 pad B7: USB_CON_D+ -> USB_CON_D-
- MX34 pad 2: unconnected-(MX34-Pad2) -> Net-(D34-A)
- R3 pad 2: Net-(C101-Pad1) -> Net-(R3-Pad2)
- R4 pad 2: Net-(C102-Pad1) -> Net-(R4-Pad2)
- SW2 pad A: Net-(C101-Pad1) -> Net-(R3-Pad2)
- SW2 pad B: Net-(C102-Pad1) -> Net-(R4-Pad2)
- U4 pad 10: COL16 -> COL4
- U4 pad 2: COL6 -> COL7
- U4 pad 3: COL5 -> COL6
- U4 pad 31: COL15 -> COL16
- U4 pad 38: COL14 -> COL15
- U4 pad 39: COL13 -> COL14
- U4 pad 4: COL4 -> COL5
- U4 pad 40: COL12 -> COL13
- U4 pad 41: COL11 -> COL12
- U4 pad 42: COL10 -> COL11
- U4 pad 43: COL9 -> COL10
- U4 pad 45: COL8 -> COL9
- U4 pad 46: COL7 -> COL8
Routing:
- net COL16: track 94.8 -> 409.2 mm, vias 5 -> 8
- net ROW0: track 296.8 -> 379.9 mm, vias 2 -> 5
- net Net-(C101-Pad1): track 45.0 -> 0.00 mm
- net Net-(C102-Pad1): track 38.3 -> 0.00 mm, vias 1 -> 0
- net Net-(R3-Pad2): track 0.00 -> 35.6 mm
- net Net-(R4-Pad2): track 0.00 -> 33.8 mm
- net +3V3: track 99.1 -> 121.5 mm
- net GND: track 73.0 -> 86.6 mm, vias 12 -> 24
- net COL4: track 146.4 -> 159.0 mm, vias 8 -> 6
- net Net-(D90-A): track 0.00 -> 9.15 mm
- net (no net): track 8.42 -> 0.00 mm
- net +5V: track 0.04 -> 8.28 mm
- net Net-(J1-CC2): track 1.64 -> 9.69 mm
- net Net-(D34-A): track 0.00 -> 7.58 mm
- net COL15: track 386.0 -> 379.9 mm
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Other:
- board text added: "3v3"
- board text added: "DFU"
- board text added: "GND"
- board text added: "MEM"
- board text added: "RST"
- board text added: "SCLK"
- board text added: "SIO"
