File: TKL_Keyboard.kicad_sch (KiCad schematic)
At the start: 214 parts, among them J1 USB_C_Receptacle_USB2.0, J2 Conn_01x05_Male, SW2 RotaryEncoder_Switch, SW3 SW_SPDT, U2 XC6206PxxxMR, U4 STM32F303C8Tx, Y1 8MHz

Commit message: small changes
Small Changes

Small Changes

Small Changes

Small Changes

Small Changes

small changes
Parts:
- added R6, R8: 10k, Resistor_SMD:R_0805_2012Metric, symbol Device:R_Small
- C1: renamed from C97; value 1uF -> 22uF; footprint Capacitor_SMD:C_0402_1005Metric -> Capacitor_SMD:C_0805_2012Metric
- C2: renamed from C98; value 1uF -> 22uF; footprint Capacitor_SMD:C_0402_1005Metric -> Capacitor_SMD:C_0805_2012Metric
- C3: renamed from C99; value 30p -> 30pF
- C4: renamed from C100; value 30p -> 30pF
- MX31: footprint MX_Only:MXOnly-1U-Hotswap -> MX_Only:MXOnly-2U-Hotswap
- Y1: value 8MHz -> 16MHz
- renumbered C105 to C10, C104 to C11, C108 to C12, C107 to C13, C101 to C14, C102 to C15, C106 to C5, C86 to C6, C94 to C7, C95 to C8, C96 to C9, R5 to R3, R6 to R4, R7 to R5, R8 to R7, SW3 to SW1
Connections:
- net +3V3: now also C12.1, FB1.1, R6.2, R8.2
- net COL10: now also U4.43 (PB7); no longer U4.42 (PB6)
- net COL11: now also U4.42 (PB6); no longer U4.41 (PB5)
- net COL12: now also U4.41 (PB5); no longer U4.40 (PB4)
- net COL13: now also U4.40 (PB4); no longer U4.39 (PB3)
- net COL14: now also U4.39 (PB3); no longer U4.38 (PA15)
- net COL15: now also U4.38 (PA15); no longer U4.31 (PA10)
- net COL16: now also U4.31 (PA10); no longer U4.10 (PA0)
- net COL4: now also U4.10 (PA0); no longer U4.4 (PC15)
- net COL5: now also U4.4 (PC15); no longer U4.3 (PC14)
- net COL6: now also U4.3 (PC14); no longer U4.2 (PC13)
- net COL7: now also U4.2 (PC13); no longer U4.46 (PB9)
- net COL8: now also U4.46 (PB9); no longer U4.45 (PB8)
- net COL9: now also U4.45 (PB8); no longer U4.43 (PB7)
- net ENCODER_A: now also C14.1
- net ENCODER_B: now also C15.1
- net GND: now also C13.1; no longer C13.2
- net NRST: now also C13.2; no longer C13.1
- net USB_CON_D+: now also J1.A6 (D+), J1.B6 (D+); no longer J1.A7 (D-), J1.B7 (D-)
- net USB_CON_D-: now also J1.A7 (D-), J1.B7 (D-); no longer J1.A6 (D+), J1.B6 (D+)
- net at R3.2, SW2.A: now also R6.1; no longer C14.1
- net at R4.2, SW2.B: now also R8.1; no longer C15.1
- net at D34.2 (A): now also MX34.2
- no-connect marks 0 -> 7
Other:
- moved on the sheet: C10, C11, C12, C13, C14, C15, C5, C6, C7, C8, C9, D10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
